File: USB_SPII2CK.kicad_sch (KiCad schematic)
At the start: 46 parts, among them J1 Conn_02x05_Odd_Even, J1 USB_B_Micro, J2 Conn_01x02, J3 Conn_01x02, J5 Conn_01x02, J6 Conn_02x08_Odd_Even, U2 FT2232HL, U2 LP2985-3.3, U3 AT93C46DN-SH-T, Y1 12.00 MHz

Commit message: Update to V1.1 (move R10 out from under connector)
Parts:
- J6: LCSC (none) -> C17282974
Changed lines of the file:
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@@
+			)
+		)
+		(property "LCSC" "C17282974"
+			(at 254 130.81 0)
+			(effects
+				(font
+					(size 1.27 1.27)
+				)
+				(hide yes)
 			)
 		)
